Commit message: imu config improvements

File: src/master_package/robots/pioneer.urdf (robot description, URDF)
Before this commit: robot pioneer3at_body, 19 links, 18 joints
Joints:
- added joint imu_joint: type fixed, parent base_link, child imu_link, origin xyz=0.3 0 0.2 rpy=0 0 0

Commit message: changes

File: src/master_package/robots/pioneer.urdf (robot description, URDF)
Before this commit: robot pioneer3at_body, 19 links, 18 joints
Links:
- link chassis: geometry collision mesh filename=file:///home/group7/Desktop/Mobile-Robots-Project/src/maste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; visual mesh filename=file:///home/group7/Desktop/Mobile-Robots-Project/src/maste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
- link laser_frame: geometry collision box size=0.01 0.01 0.01; visual mesh filename=file:///home/group7/Desktop/Mobile-Robots-Project/src/maste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
- link p3at_back_left_axle: geometry collision box size=0.01 0.01 0.01; visual mesh filename=file:///home/group7/Desktop/Mobile-Robots-Project/src/maste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
- link p3at_back_left_hub: geometry collision box size=0.01 0.01 0.01; visual mesh filename=file:///home/group7/Desktop/Mobile-Robots-Project/src/maste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
- link p3at_back_left_wheel: geometry collision mesh filename=file:///home/group7/Desktop/Mobile-Robots-Project/src/maste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; visual mesh filename=file:///home/group7/Desktop/Mobile-Robots-Project/src/maste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
- link p3at_back_right_axle: geometry collision box size=0.01 0.01 0.01; visual mesh filename=file:///home/group7/Desktop/Mobile-Robots-Project/src/maste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
- link p3at_back_right_hub: geometry collision box size=0.01 0.01 0.01; visual mesh filename=file:///home/group7/Desktop/Mobile-Robots-Project/src/maste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
- link p3at_back_right_wheel: geometry collision mesh filename=file:///home/group7/Desktop/Mobile-Robots-Project/src/maste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; visual mesh filename=file:///home/group7/Desktop/Mobile-Robots-Project/src/maste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
- link p3at_front_left_axle: geometry collision box size=0.01 0.01 0.01; visual mesh filename=file:///home/group7/Desktop/Mobile-Robots-Project/src/maste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
- link p3at_front_left_hub: geometry collision box size=0.01 0.01 0.01; visual mesh filename=file:///home/group7/Desktop/Mobile-Robots-Project/src/maste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
- link p3at_front_left_wheel: geometry collision mesh filename=file:///home/group7/Desktop/Mobile-Robots-Project/src/maste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; visual mesh filename=file:///home/group7/Desktop/Mobile-Robots-Project/src/maste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
- link p3at_front_right_axle: geometry collision box size=0.01 0.01 0.01; visual mesh filename=file:///home/group7/Desktop/Mobile-Robots-Project/src/maste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
- link p3at_front_right_hub: geometry collision box size=0.01 0.01 0.01; visual mesh filename=file:///home/group7/Desktop/Mobile-Robots-Project/src/maste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
- link p3at_front_right_wheel: geometry collision mesh filename=file:///home/group7/Desktop/Mobile-Robots-Project/src/maste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; visual mesh filename=file:///home/group7/Desktop/Mobile-Robots-Project/src/maste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
- link top_plate: geometry collision box size=0.1 0.1 0.1; visual mesh filename=file:///home/group7/Desktop/Mobile-Robots-Project/src/maste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
Joints:
- added joint imu_joint: type fixed, parent base_link, child imu_link, origin xyz=0.3 0 0.2 rpy=0 0 0

Commit message: upates_fri_17_5

File: src/master_package/robots/pioneer.urdf (robot description, URDF)
Before this commit: robot pioneer3at_body, 19 links, 19 joints
Links:
- removed link base_footprint
- removed link laser_frame
- added link cloud, mass 1e-5; collision box size=0.01 0.01 0.01; visual mesh filename=file:///src/master_package/meshes/hokuyo1.dae
- added link imu_link
- link cam_frame: geometry 
- link chassis: geometry collision mesh filename=file:///src/master_package/meshes/chassis.dae; visual mesh filename=file:///src/master_package/meshes/chassis.dae
- link p3at_back_left_axle: geometry collision box size=0.01 0.01 0.01; visual mesh filename=file:///src/master_package/meshes/p3at_meshes/axle.dae
- link p3at_back_left_hub: geometry collision box size=0.01 0.01 0.01; visual mesh filename=file:///src/master_package/meshes/p3at_meshes/right_hubcap.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
- link p3at_back_left_wheel: geometry collision mesh filename=file:///src/master_package/meshes/p3at_meshes/wheel.dae; visual mesh filename=file:///src/master_package/meshes/p3at_meshes/wheel.dae
- link p3at_back_right_axle: geometry collision box size=0.01 0.01 0.01; visual mesh filename=file:///src/master_package/meshes/p3at_meshes/axle.dae
- link p3at_back_right_hub: geometry collision box size=0.01 0.01 0.01; visual mesh filename=file:///src/master_package/meshes/p3at_meshes/right_hubcap.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
- link p3at_back_right_wheel: geometry collision mesh filename=file:///src/master_package/meshes/p3at_meshes/wheel.dae; visual mesh filename=file:///src/master_package/meshes/p3at_meshes/wheel.dae
- link p3at_front_left_axle: geometry collision box size=0.01 0.01 0.01; visual mesh filename=file:///src/master_package/meshes/p3at_meshes/axle.dae
- link p3at_front_left_hub: geometry collision box size=0.01 0.01 0.01; visual mesh filename=file:///src/master_package/meshes/p3at_meshes/left_hubcap.d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
- link p3at_front_left_wheel: geometry collision mesh filename=file:///src/master_package/meshes/p3at_meshes/wheel.dae; visual mesh filename=file:///src/master_package/meshes/p3at_meshes/wheel.dae
- link p3at_front_right_axle: geometry collision box size=0.01 0.01 0.01; visual mesh filename=file:///src/master_package/meshes/p3at_meshes/axle.dae
- link p3at_front_right_hub: geometry collision box size=0.01 0.01 0.01; visual mesh filename=file:///src/master_package/meshes/p3at_meshes/right_hubcap.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
- link p3at_front_right_wheel: geometry collision mesh filename=file:///src/master_package/meshes/p3at_meshes/wheel.dae; visual mesh filename=file:///src/master_package/meshes/p3at_meshes/wheel.dae
- link top_plate: geometry collision box size=0.1 0.1 0.1; visual mesh filename=file:///src/master_package/meshes/top.dae
Joints:
- removed joint base_joint
- joint imu_joint: parent base_link -> chassis
- joint laser_joint: child laser_frame -> cloud

Commit message: staged

File: src/master_package/robots/pioneer.urdf (robot description, URDF)
Before this commit: robot pioneer3at_body, 19 links, 18 joints
Links:
- link chassis: geometry collision mesh filename=file:///project/src/master_package/meshes/chassis.dae; visual mesh filename=file:///project/src/master_package/meshes/chassis.dae
- link cloud: geometry collision box size=0.01 0.01 0.01; visual mesh filename=file:///project/src/master_package/meshes/hokuyo1.dae
- link p3at_back_left_axle: geometry collision box size=0.01 0.01 0.01; visual mesh filename=file:///project/src/master_package/meshes/p3at_meshes/axle.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
- link p3at_back_left_hub: geometry collision box size=0.01 0.01 0.01; visual mesh filename=file:///project/src/master_package/meshes/p3at_meshes/right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
- link p3at_back_left_wheel: geometry collision mesh filename=file:///project/src/master_package/meshes/p3at_meshes/wheel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; visual mesh filename=file:///project/src/master_package/meshes/p3at_meshes/wheel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
- link p3at_back_right_axle: geometry collision box size=0.01 0.01 0.01; visual mesh filename=file:///project/src/master_package/meshes/p3at_meshes/axle.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
- link p3at_back_right_hub: geometry collision box size=0.01 0.01 0.01; visual mesh filename=file:///project/src/master_package/meshes/p3at_meshes/right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
- link p3at_back_right_wheel: geometry collision mesh filename=file:///project/src/master_package/meshes/p3at_meshes/wheel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; visual mesh filename=file:///project/src/master_package/meshes/p3at_meshes/wheel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
- link p3at_front_left_axle: geometry collision box size=0.01 0.01 0.01; visual mesh filename=file:///project/src/master_package/meshes/p3at_meshes/axle.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
- link p3at_front_left_hub: geometry collision box size=0.01 0.01 0.01; visual mesh filename=file:///project/src/master_package/meshes/p3at_meshes/left_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
- link p3at_front_left_wheel: geometry collision mesh filename=file:///project/src/master_package/meshes/p3at_meshes/wheel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; visual mesh filename=file:///project/src/master_package/meshes/p3at_meshes/wheel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
- link p3at_front_right_axle: geometry collision box size=0.01 0.01 0.01; visual mesh filename=file:///project/src/master_package/meshes/p3at_meshes/axle.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
- link p3at_front_right_hub: geometry collision box size=0.01 0.01 0.01; visual mesh filename=file:///project/src/master_package/meshes/p3at_meshes/right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
- link p3at_front_right_wheel: geometry collision mesh filename=file:///project/src/master_package/meshes/p3at_meshes/wheel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; visual mesh filename=file:///project/src/master_package/meshes/p3at_meshes/wheel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
- link top_plate: geometry collision box size=0.1 0.1 0.1; visual mesh filename=file:///project/src/master_package/meshes/top.dae
