Commit message: changes from monday night

File: src/master_package/robots/pioneer2.urdf (robot description, URDF)
Before this commit: robot pioneer3at_body, 19 links, 18 joints
Links:
- added link base_footprint
- link chassis: geometry collision mesh filename=file:///project/src/master_package/meshes/chassis.dae; visual mesh filename=file:///project/src/master_package/meshes/chassis.dae
- link cloud: geometry collision box size=0.01 0.01 0.01; visual mesh filename=file:///project/src/master_package/meshes/hokuyo1.dae
- link p3at_back_left_axle: geometry collision box size=0.01 0.01 0.01; visual mesh filename=file:///project/src/master_package/meshes/p3at_meshes/axle.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
- link p3at_back_left_hub: geometry collision box size=0.01 0.01 0.01; visual mesh filename=file:///project/src/master_package/meshes/p3at_meshes/right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
- link p3at_back_left_wheel: geometry collision mesh filename=file:///project/src/master_package/meshes/p3at_meshes/wheel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; visual mesh filename=file:///project/src/master_package/meshes/p3at_meshes/wheel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
- link p3at_back_right_axle: geometry collision box size=0.01 0.01 0.01; visual mesh filename=file:///project/src/master_package/meshes/p3at_meshes/axle.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
- link p3at_back_right_hub: geometry collision box size=0.01 0.01 0.01; visual mesh filename=file:///project/src/master_package/meshes/p3at_meshes/right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
- link p3at_back_right_wheel: geometry collision mesh filename=file:///project/src/master_package/meshes/p3at_meshes/wheel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; visual mesh filename=file:///project/src/master_package/meshes/p3at_meshes/wheel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
- link p3at_front_left_axle: geometry collision box size=0.01 0.01 0.01; visual mesh filename=file:///project/src/master_package/meshes/p3at_meshes/axle.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
- link p3at_front_left_hub: geometry collision box size=0.01 0.01 0.01; visual mesh filename=file:///project/src/master_package/meshes/p3at_meshes/left_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
- link p3at_front_left_wheel: geometry collision mesh filename=file:///project/src/master_package/meshes/p3at_meshes/wheel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; visual mesh filename=file:///project/src/master_package/meshes/p3at_meshes/wheel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
- link p3at_front_right_axle: geometry collision box size=0.01 0.01 0.01; visual mesh filename=file:///project/src/master_package/meshes/p3at_meshes/axle.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
- link p3at_front_right_hub: geometry collision box size=0.01 0.01 0.01; visual mesh filename=file:///project/src/master_package/meshes/p3at_meshes/right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
- link p3at_front_right_wheel: geometry collision mesh filename=file:///project/src/master_package/meshes/p3at_meshes/wheel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; visual mesh filename=file:///project/src/master_package/meshes/p3at_meshes/wheel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
- link top_plate: geometry collision box size=0.1 0.1 0.1; visual mesh filename=file:///project/src/master_package/meshes/top.dae
Joints:
- added joint base_joint: type fixed, parent base_link, child base_footprint, origin xyz=0.0 0.0 0.0 rpy=0 0 0
